Commit message: added more bodycams

File: src/curobo/content/assets/robot/ur_description/ur5e_bodycams.urdf (robot description, URDF)
Before this commit: robot ur5e_robot, 17 links, 16 joints
Links:
- added link cam7_link
- added link cam8_link
Joints:
- added joint cam7_joint: type fixed, parent forearm_link, child cam7_link, origin xyz=-0.2040509 -0.038 0.005 rpy=1.5707963267948966 0 3.141592653589793
- added joint cam8_joint: type fixed, parent forearm_link, child cam8_link, origin xyz=-0.2040509 +0.038 0.005 rpy=1.5707963267948966 0 0
